Commit message: new branch: simulation for actions unit in course ROS2 basics

File: leo_rover_simulation/leo_description/urdf/macros.xacro (robot description, xacro)
@@ -176,5 +176,5 @@
       <child link="${link_prefix}rocker_L_link"/>
       <axis xyz="0 1 0"/>
-      <limit effort="100.0" lower="-0.24" upper="0.24" velocity="100.0"/>
+      <limit effort="100.0" lower="-0.01" upper="0.01" velocity="100.0"/>
       <dynamics friction="1.0" damping="0.1"/>
     </joint>
@@ -184,5 +184,5 @@
       <child link="${link_prefix}rocker_R_link"/>
       <axis xyz="0 1 0"/>
-      <limit effort="100.0" lower="-0.24" upper="0.24" velocity="100.0"/>
+      <limit effort="100.0" lower="-0.01" upper="0.01" velocity="100.0"/>
       <dynamics friction="1.0" damping="0.1"/>
       <mimic joint="rocker_L_joint"/>
@@ -453,5 +453,5 @@
     </gazebo>
     <!-- rocker differential -->
-    <gazebo>
+    <!-- <gazebo>
       <plugin name="leo_gz_DifferentialSystem" filename="libleo_gazebo_differential_plugin.so">
         <jointA>rocker_L_joint</jointA>
@@ -464,5 +464,5 @@
         <forceConstant>100.0</forceConstant>
       </plugin>
-    </gazebo>
+    </gazebo> -->
     <gazebo reference="${link_prefix}imu_frame">
       <sensor type="imu" name="leo_imu_sensor">
@@ -475,17 +475,36 @@
     </gazebo>
     <gazebo>
+        <plugin name="four_diff_controller" filename="libgazebo_ros_diff_drive.so">
+            <update_rate>30</update_rate>
+            <num_wheel_pairs>2</num_wheel_pairs>
+            <left_joint>wheel_FL_joint</left_joint>
+            <right_joint>wheel_FR_joint</right_joint>
+            <left_joint>wheel_RL_joint</left_joint>
+            <right_joint>wheel_RR_joint</right_joint>
+            <wheel_separation>0.358</wheel_separation>
+            <wheel_diameter>0.13</wheel_diameter>
+            <max_wheel_torque>20</max_wheel_torque>
+            <max_wheel_acceleration>1.0</max_wheel_acceleration>
+            <command_topic>cmd_vel</command_topic>
+            <publish_odom>true</publish_odom>
+            <publish_odom_tf>true</publish_odom_tf>
+            <publish_wheel_tf>true</publish_wheel_tf>
+            <odometry_topic>odom</odometry_topic>
+            <odometry_frame>odom</odometry_frame>
+            <robot_base_frame>base_footprint</robot_base_frame>
+            <odometry_source>1</odometry_source>
+        </plugin>
+    </gazebo>
+    <!-- <gazebo>
       <plugin filename="libgazebo_ros_diff_drive.so" name="four_diff_controller">
         <left_joint>wheel_FL_joint</left_joint>
         <right_joint>wheel_FR_joint</right_joint>
-        <!-- kinematics -->
         <wheel_separation>0.358</wheel_separation>
         <wheel_diameter>0.13</wheel_diameter>
-        <!-- limits -->
         <max_wheel_torque>20</max_wheel_torque>
         <max_wheel_acceleration>1.0</max_wheel_acceleration>
-        <!-- output -->
         <publish_odom>true</publish_odom>
         <publish_odom_tf>true</publish_odom_tf>
-        <publish_wheel_tf>false</publish_wheel_tf>
+        <publish_wheel_tf>true</publish_wheel_tf>
         <odometry_topic>odom</odometry_topic>
         <odometry_frame>odom</odometry_frame>
@@ -493,7 +512,4 @@
         <odometry_source>1</odometry_source>
         <command_topic>cmd_vel</command_topic>
-        <ros>
-            <!-- <remapping>odom:=/odometry</remapping> -->
-        </ros>
       </plugin>
     </gazebo>
@@ -502,14 +518,11 @@
         <left_joint>wheel_RL_joint</left_joint>
         <right_joint>wheel_RR_joint</right_joint>
-        <!-- kinematics -->
         <wheel_separation>0.358</wheel_separation>
         <wheel_diameter>0.13</wheel_diameter>
-        <!-- limits -->
         <max_wheel_torque>20</max_wheel_torque>
         <max_wheel_acceleration>1.0</max_wheel_acceleration>
-        <!-- output -->
-        <publish_odom>true</publish_odom>
+        <publish_odom>false</publish_odom>
         <publish_odom_tf>true</publish_odom_tf>
-        <publish_wheel_tf>false</publish_wheel_tf>
+        <publish_wheel_tf>true</publish_wheel_tf>
         <odometry_topic>odom</odometry_topic>
         <odometry_frame>odom</odometry_frame>
@@ -517,9 +530,6 @@
         <odometry_source>1</odometry_source>
         <command_topic>cmd_vel</command_topic>
-        <ros>
-            <!-- <remapping>odom:=/odometry</remapping> -->
-        </ros>
       </plugin>
-    </gazebo>
+    </gazebo> -->
   </xacro:macro>
   <xacro:macro name="leo_sim"

File: leo_rover_simulation/leo_description/urdf/sensors.xacro (robot description, xacro)
@@ -2,6 +2,6 @@
 <robot xmlns:xacro="http://www.ros.org/wiki/xacro">
   <xacro:macro name="laser_scan" params="robot_name parent_name origin_xyz sensor_YAW">
-      <link name="${robot_name}_laser_scan_model_link">
-        <visual name="${robot_name}_visual_laser_scan_link">
+      <link name="${robot_name}lidar_1_link">
+        <visual name="${robot_name}visual_lidar_1_link">
           <origin rpy="0 0 0" xyz="0 0 0"/>
           <geometry>
@@ -9,5 +9,5 @@
           </geometry>
         </visual>
-        <collision name="${robot_name}_collision_laser_scan_link">
+        <collision name="${robot_name}collision_lidar_1_link">
           <origin rpy="0 0 0" xyz="0 0 0.0098125"/>
           <geometry>
@@ -21,23 +21,16 @@
         </inertial>
       </link>
-    <joint name="${robot_name}_laser_scan_model_link_joint" type="fixed">
+    <joint name="${robot_name}laser_1_joint" type="fixed">
         <origin xyz="${origin_xyz}" rpy="0 0 ${sensor_YAW}" />
         <parent link="${parent_name}" />
-        <child link="${robot_name}_laser_scan_model_link" />
+        <child link="${robot_name}lidar_1_link" />
     </joint>
-    <link name="${robot_name}_laser_scan_frame">
-    </link>
-    <joint name="${robot_name}_laser_scan_frame_joint" type="fixed">
-        <origin xyz="0 0 0.03" rpy="0 0 ${sensor_YAW}" />
-        <parent link="${robot_name}_laser_scan_model_link" />
-        <child link="${robot_name}_laser_scan_frame" />
-    </joint>
-    <gazebo reference="${robot_name}_laser_scan_frame">
-      <sensor name="sensor_ray" type="ray">
+    <gazebo reference="${robot_name}lidar_1_link">
+      <sensor name="lidar_1_sensor" type="ray">
           <pose>0 0 0 0 0 0</pose>
           <ray>
             <scan>
               <horizontal>
-                <samples>200</samples>
+                <samples>100</samples>
                 <resolution>1.0</resolution>
                 <min_angle>-2.2</min_angle>
@@ -46,5 +39,5 @@
             </scan>
             <range>
-              <min>0.1</min>
+              <min>0.3</min>
               <max>20.0</max>
             </range>
@@ -53,10 +46,10 @@
           <visualize>true</visualize>
           <update_rate>10.0</update_rate>
-          <plugin name="laser" filename="libgazebo_ros_ray_sensor.so">
+          <plugin name="lidar_1" filename="libgazebo_ros_ray_sensor.so">
             <ros>
               <namespace>${robot_name}</namespace>
-              <remapping>~/out:=laser_scan</remapping>
+              <remapping>~/out:=/scan</remapping>
             </ros>
-            <frame_name>${robot_name}_laser_scan_frame</frame_name>
+            <frame_name>${robot_name}lidar_1_link</frame_name>
             <output_type>sensor_msgs/LaserScan</output_type>
           </plugin>

Commit message: Add: Rover default behaviour and files together with Actions Rover

File: leo_rover_simulation/leo_description/urdf/macros.xacro (robot description, xacro)
@@ -176,5 +176,5 @@
       <child link="${link_prefix}rocker_L_link"/>
       <axis xyz="0 1 0"/>
-      <limit effort="100.0" lower="-0.01" upper="0.01" velocity="100.0"/>
+      <limit effort="100.0" lower="-0.24" upper="0.24" velocity="100.0"/>
       <dynamics friction="1.0" damping="0.1"/>
     </joint>
@@ -184,5 +184,5 @@
       <child link="${link_prefix}rocker_R_link"/>
       <axis xyz="0 1 0"/>
-      <limit effort="100.0" lower="-0.01" upper="0.01" velocity="100.0"/>
+      <limit effort="100.0" lower="-0.24" upper="0.24" velocity="100.0"/>
       <dynamics friction="1.0" damping="0.1"/>
       <mimic joint="rocker_L_joint"/>
@@ -453,5 +453,5 @@
     </gazebo>
     <!-- rocker differential -->
-    <!-- <gazebo>
+    <gazebo>
       <plugin name="leo_gz_DifferentialSystem" filename="libleo_gazebo_differential_plugin.so">
         <jointA>rocker_L_joint</jointA>
@@ -464,5 +464,5 @@
         <forceConstant>100.0</forceConstant>
       </plugin>
-    </gazebo> -->
+    </gazebo>
     <gazebo reference="${link_prefix}imu_frame">
       <sensor type="imu" name="leo_imu_sensor">
@@ -475,36 +475,17 @@
     </gazebo>
     <gazebo>
-        <plugin name="four_diff_controller" filename="libgazebo_ros_diff_drive.so">
-            <update_rate>30</update_rate>
-            <num_wheel_pairs>2</num_wheel_pairs>
-            <left_joint>wheel_FL_joint</left_joint>
-            <right_joint>wheel_FR_joint</right_joint>
-            <left_joint>wheel_RL_joint</left_joint>
-            <right_joint>wheel_RR_joint</right_joint>
-            <wheel_separation>0.358</wheel_separation>
-            <wheel_diameter>0.13</wheel_diameter>
-            <max_wheel_torque>20</max_wheel_torque>
-            <max_wheel_acceleration>1.0</max_wheel_acceleration>
-            <command_topic>cmd_vel</command_topic>
-            <publish_odom>true</publish_odom>
-            <publish_odom_tf>true</publish_odom_tf>
-            <publish_wheel_tf>true</publish_wheel_tf>
-            <odometry_topic>odom</odometry_topic>
-            <odometry_frame>odom</odometry_frame>
-            <robot_base_frame>base_footprint</robot_base_frame>
-            <odometry_source>1</odometry_source>
-        </plugin>
-    </gazebo>
-    <!-- <gazebo>
       <plugin filename="libgazebo_ros_diff_drive.so" name="four_diff_controller">
         <left_joint>wheel_FL_joint</left_joint>
         <right_joint>wheel_FR_joint</right_joint>
+        <!-- kinematics -->
         <wheel_separation>0.358</wheel_separation>
         <wheel_diameter>0.13</wheel_diameter>
+        <!-- limits -->
         <max_wheel_torque>20</max_wheel_torque>
         <max_wheel_acceleration>1.0</max_wheel_acceleration>
+        <!-- output -->
         <publish_odom>true</publish_odom>
         <publish_odom_tf>true</publish_odom_tf>
-        <publish_wheel_tf>true</publish_wheel_tf>
+        <publish_wheel_tf>false</publish_wheel_tf>
         <odometry_topic>odom</odometry_topic>
         <odometry_frame>odom</odometry_frame>
@@ -512,4 +493,7 @@
         <odometry_source>1</odometry_source>
         <command_topic>cmd_vel</command_topic>
+        <ros>
+            <!-- <remapping>odom:=/odometry</remapping> -->
+        </ros>
       </plugin>
     </gazebo>
@@ -518,11 +502,14 @@
         <left_joint>wheel_RL_joint</left_joint>
         <right_joint>wheel_RR_joint</right_joint>
+        <!-- kinematics -->
         <wheel_separation>0.358</wheel_separation>
         <wheel_diameter>0.13</wheel_diameter>
+        <!-- limits -->
         <max_wheel_torque>20</max_wheel_torque>
         <max_wheel_acceleration>1.0</max_wheel_acceleration>
-        <publish_odom>false</publish_odom>
+        <!-- output -->
+        <publish_odom>true</publish_odom>
         <publish_odom_tf>true</publish_odom_tf>
-        <publish_wheel_tf>true</publish_wheel_tf>
+        <publish_wheel_tf>false</publish_wheel_tf>
         <odometry_topic>odom</odometry_topic>
         <odometry_frame>odom</odometry_frame>
@@ -530,6 +517,9 @@
         <odometry_source>1</odometry_source>
         <command_topic>cmd_vel</command_topic>
+        <ros>
+            <!-- <remapping>odom:=/odometry</remapping> -->
+        </ros>
       </plugin>
-    </gazebo> -->
+    </gazebo>
   </xacro:macro>
   <xacro:macro name="leo_sim"

File: leo_rover_simulation/leo_description/urdf/sensors.xacro (robot description, xacro)
@@ -2,6 +2,6 @@
 <robot xmlns:xacro="http://www.ros.org/wiki/xacro">
   <xacro:macro name="laser_scan" params="robot_name parent_name origin_xyz sensor_YAW">
-      <link name="${robot_name}lidar_1_link">
-        <visual name="${robot_name}visual_lidar_1_link">
+      <link name="${robot_name}_laser_scan_model_link">
+        <visual name="${robot_name}_visual_laser_scan_link">
           <origin rpy="0 0 0" xyz="0 0 0"/>
           <geometry>
@@ -9,5 +9,5 @@
           </geometry>
         </visual>
-        <collision name="${robot_name}collision_lidar_1_link">
+        <collision name="${robot_name}_collision_laser_scan_link">
           <origin rpy="0 0 0" xyz="0 0 0.0098125"/>
           <geometry>
@@ -21,16 +21,23 @@
         </inertial>
       </link>
-    <joint name="${robot_name}laser_1_joint" type="fixed">
+    <joint name="${robot_name}_laser_scan_model_link_joint" type="fixed">
         <origin xyz="${origin_xyz}" rpy="0 0 ${sensor_YAW}" />
         <parent link="${parent_name}" />
-        <child link="${robot_name}lidar_1_link" />
+        <child link="${robot_name}_laser_scan_model_link" />
     </joint>
-    <gazebo reference="${robot_name}lidar_1_link">
-      <sensor name="lidar_1_sensor" type="ray">
+    <link name="${robot_name}_laser_scan_frame">
+    </link>
+    <joint name="${robot_name}_laser_scan_frame_joint" type="fixed">
+        <origin xyz="0 0 0.03" rpy="0 0 ${sensor_YAW}" />
+        <parent link="${robot_name}_laser_scan_model_link" />
+        <child link="${robot_name}_laser_scan_frame" />
+    </joint>
+    <gazebo reference="${robot_name}_laser_scan_frame">
+      <sensor name="sensor_ray" type="ray">
           <pose>0 0 0 0 0 0</pose>
           <ray>
             <scan>
               <horizontal>
-                <samples>100</samples>
+                <samples>200</samples>
                 <resolution>1.0</resolution>
                 <min_angle>-2.2</min_angle>
@@ -39,5 +46,5 @@
             </scan>
             <range>
-              <min>0.3</min>
+              <min>0.1</min>
               <max>20.0</max>
             </range>
@@ -46,10 +53,10 @@
           <visualize>true</visualize>
           <update_rate>10.0</update_rate>
-          <plugin name="lidar_1" filename="libgazebo_ros_ray_sensor.so">
+          <plugin name="laser" filename="libgazebo_ros_ray_sensor.so">
             <ros>
               <namespace>${robot_name}</namespace>
-              <remapping>~/out:=/scan</remapping>
+              <remapping>~/out:=laser_scan</remapping>
             </ros>
-            <frame_name>${robot_name}lidar_1_link</frame_name>
+            <frame_name>${robot_name}_laser_scan_frame</frame_name>
             <output_type>sensor_msgs/LaserScan</output_type>
           </plugin>
